File: PCB/main-board/main-board/main-board.kicad_sch (KiCad schematic)
At the start: 18 parts, among them Q1 PN2222A, Q2 IRLIZ44N, SW1 RotaryEncoder_Switch_MP, U1 LM358, U2 L7805

Commit message: update
Parts:
- added J1: Power Input, symbol Connector:Screw_Terminal_01x02
- added J2: Screw_Terminal_01x02, symbol Connector:Screw_Terminal_01x02
- added J3: Screw_Terminal_01x03, symbol Connector:Screw_Terminal_01x03
Connections:
- net GND: now also J1.1 (Pin_1)
- new net +24V: J1.2 (Pin_2)
