File: PCB/main-board/main-board.kicad_sch (KiCad schematic)
At the start: 21 parts, among them J1 Power Input, J2 Screw_Terminal_01x02, J3 Screw_Terminal_01x03, Q1 PN2222A, Q2 IRLIZ44N, SW1 RotaryEncoder_Switch_MP, U1 LM358, U2 L7805

Commit message: updated KiCad files
Parts:
- added C10: 100nF, symbol Device:C
- added C111: 330nF, symbol Device:C
- added C12: 10uf 35v, symbol Device:C_Polarized_US
- added C13: 10µF, symbol Device:C_Polarized_US
- added C8: 2nF, symbol Device:C
- added D4: 1N4007, Diode_THT:D_DO-41_SOD81_P10.16mm_Horizontal, symbol Diode:1N4007
- added R11, R7: 10K, symbol Device:R
- added R8, R9: 200K, symbol Device:R
- added R9: 1K, symbol Device:R
- U1: footprint Package_TO_SOT_THT:TO-99-8 -> Package_DIP:DIP-8_W7.62mm
Connections:
- net +24V: now also U2.1 (IN), C12.1
- net GND: now also U2.2 (GND), C13.2, C8.2, D4.1 (K), R9.1
- net A0: now reaches A1.19 (A0)
- net A0: now also R8.1
- net A1: now reaches A1.20 (A1)
- new net: C13.1, C8.1, D4.2 (A), R7.2, R8.2, R9.2
- new net P+: R7.1
- no-connect marks 20 -> 18
Other:
- moved on the sheet: U2
