File: PCB/main-board/main-board.kicad_sch (KiCad schematic)
At the start: 33 parts, among them J1 Conn_01x02_Pin, Q1 PN2222A, SW1 RotaryEncoder_Switch_MP, U1 LM358, U2 IRLIZ44N, U3 L7805

Commit message: updated PCB files
Parts:
- removed C10: 100nF, Capacitor_SMD:C_0402_1005Metric, symbol Device:C
- removed C11: 330nF, Capacitor_SMD:C_0603_1608Metric, symbol Device:C
- removed C12: 10uf 35v, Capacitor_SMD:CP_Elec_5x4.4, symbol Device:C_Polarized_US
- removed U3: L7805, Package_TO_SOT_THT:TO-220F-3_Vertical, symbol Regulator_Linear:L7805
- added C3: 100nf, Capacitor_SMD:C_0402_1005Metric, symbol Device:C
- added C4, C5: 220uf, Capacitor_SMD:CP_Elec_8x10, symbol Device:C_Polarized_US
- added D5, D7: 1N4007, Diode_THT:D_DO-41_SOD81_P10.16mm_Horizontal, symbol Diode:1N4007
- added D6: B120-E3, Diode_SMD:D_SMA, symbol Diode:B120-E3
- added L1: L_Small, symbol Device:L_Small
- added U3: LM2596S-5, Package_TO_SOT_SMD:TO-263-5_TabPin3, symbol Regulator_Switching:LM2596S-5
Connections:
- net GND: now also C3.2, C4.2, C5.2, D6.2 (A), U3.3 (GND), U3.5 (~{ON}/OFF)
- net VCC: now also D7.1 (K), U3.4 (FB)
- net 24V+ renamed +24V
- net +24V: now also D5.2 (A)
- new net: C3.1, C5.1, D5.1 (K), U3.1 (VIN)
- new net: D6.1 (K), L1.1, U3.2 (OUT)
- new net: C4.1, D7.2 (A), L1.2
Other:
- moved on the sheet: A1, BZ1, Brd1, C1, C13, C7, C8, D1, D2, D3, D4, Iron_conect1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

Commit message: update
Parts:
- Brd1: footprint (none) -> library:128x64OLED
- C8: footprint (none) -> Capacitor_SMD:C_0402_1005Metric
- D5, D7: footprint Diode_THT:D_DO-41_SOD81_P10.16mm_Horizontal -> Diode_SMD:D_SOD-123
- L1: value L_Small -> 330uH; footprint (none) -> Inductor_SMD:L_Coilcraft_LPS3314
- U1: footprint (none) -> Package_SO:TSSOP-8_3x3mm_P0.65mm
Other:
- moved on the sheet: D5, D6, U3

Commit message: update
Parts:
- Brd1: footprint library:128x64OLED -> SSD1306:128x64OLED
Changed lines of the file:
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@@
 	(label "SCL"
 		(at 81.28 69.85 0)
-		(fields_autoplaced yes)
 		(effects
 			(font
@@
 	(label "SDA"
 		(at 81.28 67.31 0)
-		(fields_autoplaced yes)
 		(effects
 			(font
@@
 	(label "SDA"
 		(at 193.04 77.47 270)
-		(fields_autoplaced yes)
 		(effects
 			(font
@@
 	(label "SCL"
 		(at 204.47 77.47 270)
-		(fields_autoplaced yes)
 		(effects
 			(font
@@
 			)
 		)
-		(property "Footprint" "library:128x64OLED"
+		(property "Footprint" "SSD1306:128x64OLED"
 			(at 196.85 60.96 0)
 			(effects

Commit message: update
Parts:
- Brd1: footprint SSD1306:128x64OLED -> library:128x64OLED
- C13: value 10µF -> 10uf 35V
- C4: footprint Capacitor_SMD:CP_Elec_8x10 -> Battery:BatteryHolder_ComfortableElectronic_CH273-2450_1x2450
- Q1: value PN2222A -> 2N2222A
Other:
- moved on the sheet: D2
Changed lines of the file:
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@@
 	(wire
 		(pts
+			(xy 118.11 44.45) (xy 118.11 43.18)
+		)
+		(stroke
+			(width 0)
+			(type default)
+		)
+	)
+	(wire
+		(pts
 			(xy 175.26 48.26) (xy 175.26 54.61)
 		)
@@
 	(wire
 		(pts
+			(xy 118.11 52.07) (xy 118.11 50.8)
+		)
+		(stroke
+			(width 0)
+			(type default)
+		)
+	)
+	(wire
+		(pts
 			(xy 147.32 38.1) (xy 139.7 38.1)
 		)
@@
 			(effects
 				(font
-					(size 0.6 0.6)
+					(size 1 1)
 				)
 				(justify left)
@@
 			(effects
 				(font
-					(size 0.6 0.6)
+					(size 1 1)
 				)
 				(justify left)
@@
 	(symbol
 		(lib_id "Diode:1N4007")
-		(at 118.11 46.99 90)
+		(at 118.11 48.26 90)
 		(unit 1)
 		(exclude_from_sim no)
@@
 		(fields_autoplaced yes)
 		(property "Reference" "D2"
-			(at 120.65 45.7199 90)
+			(at 120.65 46.9899 90)
 			(effects
 				(font
@@
 		)
 		(property "Value" "1N4007"
-			(at 120.65 48.2599 90)
+			(at 120.65 49.5299 90)
 			(effects
 				(font
@@
 		)
 		(property "Footprint" "Diode_SMD:D_SOD-123"
-			(at 122.555 46.99 0)
+			(at 122.555 48.26 0)
 			(effects
 				(font
@@
 		)
 		(property "Datasheet" "http://www.vishay.com/docs/88503/1n4001.pdf"
-			(at 118.11 46.99 0)
+			(at 118.11 48.26 0)
 			(effects
 				(font
@@
 		)
 		(property "Description" "1000V 1A General Purpose Rectifier Diode, DO-41"
-			(at 118.11 46.99 0)
+			(at 118.11 48.26 0)
 			(effects
 				(font
@@
 		)
 		(property "Sim.Device" "D"
-			(at 118.11 46.99 0)
+			(at 118.11 48.26 0)
 			(effects
 				(font
@@
 		)
 		(property "Sim.Pins" "1=K 2=A"
-			(at 118.11 46.99 0)
+			(at 118.11 48.26 0)
 			(effects
 				(font
@@
 			(effects
 				(font
-					(size 1.27 1.27)
+					(size 1 1)
 				)
 				(justify left)
@@
 			(effects
 				(font
-					(size 1.27 1.27)
+					(size 1 1)
 				)
 				(justify left)
@@
 		(on_board yes)
 		(dnp no)
-		(fields_autoplaced yes)
 		(property "Reference" "C13"
-			(at 111.76 46.3549 0)
+			(at 99.568 47.752 0)
 			(effects
 				(font
-					(size 1.27 1.27)
+					(size 1 1)
 				)
 				(justify left)
 			)
 		)
-		(property "Value" "10µF"
-			(at 111.76 48.8949 0)
+		(property "Value" "10uf 35V"
+			(at 97.536 49.53 0)
 			(effects
 				(font
-					(size 1.27 1.27)
+					(size 1 1)
 				)
 				(justify left)
@@
 		(on_board yes)
 		(dnp no)
-		(fields_autoplaced yes)
 		(property "Reference" "Brd1"
 			(at 204.47 53.3399 0)
@@
 			)
 		)
-		(property "Footprint" "SSD1306:128x64OLED"
-			(at 196.85 60.96 0)
+		(property "Footprint" "library:128x64OLED"
+			(at 197.612 56.896 0)
 			(effects
 				(font
@@
 			)
 		)
-		(property "Value" "PN2222A"
+		(property "Value" "2N2222A"
 			(at 54.61 142.2399 0)
 			(effects
@@
 			)
 		)
-		(property "Footprint" "Capacitor_SMD:CP_Elec_8x10"
+		(property "Footprint" "Battery:BatteryHolder_ComfortableElectronic_CH273-2450_1x2450"
 			(at 201.93 125.73 0)
 			(effects

Commit message: update
Parts:
- C1, C3, C8: footprint Capacitor_SMD:C_0402_1005Metric -> Capacitor_SMD:C_1206_3216Metric
- C13, C7: footprint Capacitor_SMD:CP_Elec_5x4.4 -> Capacitor_SMD:CP_Elec_5x5.7
- C4: footprint Battery:BatteryHolder_ComfortableElectronic_CH273-2450_1x2450 -> Capacitor_SMD:CP_Elec_8x10
- D2, D5, D7: footprint Diode_SMD:D_SOD-123 -> Diode_SMD:D_SMA
- D6: value B120-E3 -> SS34
- L1: footprint Inductor_SMD:L_Coilcraft_LPS3314 -> Inductor_SMD:L_Coilcraft_LPS4414
- Q1: footprint Package_TO_SOT_THT:TO-92_Wide -> Package_TO_SOT_SMD:SOT-23_Handsoldering
- R1, R11, R14, R3, R4, R6, R7: footprint Resistor_SMD:R_0201_0603Metric -> Resistor_SMD:R_1206_3216Metric
- R12: footprint Resistor_SMD:R_0805_2012Metric -> Resistor_SMD:R_1206_3216Metric
- R13: footprint Resistor_SMD:R_0603_1608Metric -> Resistor_SMD:R_1206_3216Metric
- R5, R8, R9: footprint Resistor_SMD:R_0402_1005Metric -> Resistor_SMD:R_1206_3216Metric
Changed lines of the file:
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@@
 			)
 		)
-		(property "Footprint" "Capacitor_SMD:C_0402_1005Metric"
+		(property "Footprint" "Capacitor_SMD:C_1206_3216Metric"
 			(at 136.8552 127 0)
 			(effects
@@
 			)
 		)
-		(property "Footprint" "Resistor_SMD:R_0201_0603Metric"
+		(property "Footprint" "Resistor_SMD:R_1206_3216Metric"
 			(at 170.18 43.688 90)
 			(effects
@@
 			)
 		)
-		(property "Footprint" "Resistor_SMD:R_0603_1608Metric"
+		(property "Footprint" "Resistor_SMD:R_1206_3216Metric"
 			(at 140.208 87.63 90)
 			(effects
@@
 			)
 		)
-		(property "Footprint" "Capacitor_SMD:C_0402_1005Metric"
+		(property "Footprint" "Capacitor_SMD:C_1206_3216Metric"
 			(at 131.7752 50.8 0)
 			(effects
@@
 			)
 		)
-		(property "Value" "B120-E3"
+		(property "Value" "SS34"
 			(at 177.8 126.6824 90)
 			(effects
@@
 			)
 		)
-		(property "Footprint" "Diode_SMD:D_SOD-123"
+		(property "Footprint" "Diode_SMD:D_SMA"
 			(at 122.555 48.26 0)
 			(effects
@@
 			)
 		)
-		(property "Footprint" "Capacitor_SMD:C_0402_1005Metric"
+		(property "Footprint" "Capacitor_SMD:C_1206_3216Metric"
 			(at 176.2252 62.23 0)
 			(effects
@@
 			)
 		)
-		(property "Footprint" "Diode_SMD:D_SOD-123"
+		(property "Footprint" "Diode_SMD:D_SMA"
 			(at 187.325 113.03 0)
 			(effects
@@
 			)
 		)
-		(property "Footprint" "Resistor_SMD:R_0201_0603Metric"
+		(property "Footprint" "Resistor_SMD:R_1206_3216Metric"
 			(at 31.75 139.192 90)
 			(effects
@@
 			)
 		)
-		(property "Footprint" "Capacitor_SMD:CP_Elec_5x4.4"
+		(property "Footprint" "Capacitor_SMD:CP_Elec_5x5.7"
 			(at 107.95 48.26 0)
 			(effects
@@
 			)
 		)
-		(property "Footprint" "Resistor_SMD:R_0805_2012Metric"
+		(property "Footprint" "Resistor_SMD:R_1206_3216Metric"
 			(at 147.32 79.502 90)
 			(effects
@@
 			)
 		)
-		(property "Footprint" "Resistor_SMD:R_0201_0603Metric"
+		(property "Footprint" "Resistor_SMD:R_1206_3216Metric"
 			(at 229.87 29.718 90)
 			(effects
@@
 			)
 		)
-		(property "Footprint" "Resistor_SMD:R_0201_0603Metric"
+		(property "Footprint" "Resistor_SMD:R_1206_3216Metric"
 			(at 207.772 69.85 90)
 			(effects
@@
 			)
 		)
-		(property "Footprint" "Resistor_SMD:R_0402_1005Metric"
+		(property "Footprint" "Resistor_SMD:R_1206_3216Metric"
 			(at 133.35 34.798 90)
 			(effects
@@
 			)
 		)
-		(property "Footprint" "Resistor_SMD:R_0201_0603Metric"
+		(property "Footprint" "Resistor_SMD:R_1206_3216Metric"
 			(at 104.14 44.958 90)
 			(effects
@@
 			)
 		)
-		(property "Footprint" "Resistor_SMD:R_0402_1005Metric"
+		(property "Footprint" "Resistor_SMD:R_1206_3216Metric"
 			(at 141.478 46.99 90)
 			(effects
@@
 			)
 		)
-		(property "Footprint" "Diode_SMD:D_SOD-123"
+		(property "Footprint" "Diode_SMD:D_SMA"
 			(at 119.38 112.395 0)
 			(effects
@@
 			)
 		)
-		(property "Footprint" "Capacitor_SMD:CP_Elec_5x4.4"
+		(property "Footprint" "Capacitor_SMD:CP_Elec_5x5.7"
 			(at 54.61 160.02 0)
 			(effects
@@
 			)
 		)
-		(property "Footprint" "Resistor_SMD:R_0201_0603Metric"
+		(property "Footprint" "Resistor_SMD:R_1206_3216Metric"
 			(at 203.962 69.85 90)
 			(effects
@@
 			)
 		)
-		(property "Footprint" "Package_TO_SOT_THT:TO-92_Wide"
+		(property "Footprint" "Package_TO_SOT_SMD:SOT-23_Handsoldering"
 			(at 54.61 142.875 0)
 			(effects
@@
 			)
 		)
-		(property "Footprint" "Resistor_SMD:R_0201_0603Metric"
+		(property "Footprint" "Resistor_SMD:R_1206_3216Metric"
 			(at 164.592 58.42 90)
 			(effects
@@
 			)
 		)
-		(property "Footprint" "Battery:BatteryHolder_ComfortableElectronic_CH273-2450_1x2450"
+		(property "Footprint" "Capacitor_SMD:CP_Elec_8x10"
 			(at 201.93 125.73 0)
 			(effects
@@
 			)
 		)
-		(property "Footprint" "Inductor_SMD:L_Coilcraft_LPS3314"
+		(property "Footprint" "Inductor_SMD:L_Coilcraft_LPS4414"
 			(at 185.42 121.92 0)
 			(effects
@@
 			)
 		)
-		(property "Footprint" "Resistor_SMD:R_0402_1005Metric"
+		(property "Footprint" "Resistor_SMD:R_1206_3216Metric"
 			(at 43.18 130.048 90)
 			(effects
