File: PCB/main-board/main-board.kicad_pcb (KiCad board)
At the start: 2 copper layers, 39 parts, among them J1 Conn_01x02_Pin, Q1 PN2222A, SW1 RotaryEncoder_Switch_MP, U1 LM358, U2 IRLIZ44N, U3 L7805

Commit message: update
Parts:
- removed C10 (x2): 100nF, Capacitor_SMD:C_0402_1005Metric
- removed C11: 330nF, Capacitor_SMD:C_0603_1608Metric
- removed C12 (x2): 10uf 35v, Capacitor_SMD:CP_Elec_5x4.4
- removed the C13 at (139.8, 119.0)
- removed the C13 at (91.3, 87.5)
- removed the C7 at (165.3, 58.0)
- removed the C7 at (92.3, 65.0)
- removed the D1 at (137.4, 74.7)
- removed the D1 at (128.0, 63.5)
- removed the D2 at (79.7, 96.5)
- removed the D2 at (88.5, 59.3)
- removed the D3 at (157.5, 69.0)
- removed the D3 at (116.2, 81.6)
- added Brd1: SSD1306, library:128x64OLED, F.Cu at (140.9, 79.3)
- added C13: 10µF, Capacitor_SMD:CP_Elec_5x4.4, F.Cu at (137.9, 60.7)
- added C3: 100nf, Capacitor_SMD:C_0402_1005Metric, F.Cu at (171.0, 112.5)
- added C4: 220uf, Capacitor_SMD:CP_Elec_8x10, F.Cu at (152.0, 101.0)
- added C5: 220uf, Capacitor_SMD:CP_Elec_8x10, F.Cu at (152.0, 110.8)
- added C7: 10uf 35V, Capacitor_SMD:CP_Elec_5x4.4, F.Cu at (118.3, 109.6)
- added D1: 1N5819, Diode_SMD:D_SOD-123, F.Cu at (145.9, 55.6)
- added D2: 1N4007, Diode_SMD:D_SOD-123, F.Cu at (149.2, 55.6)
- added D3: 5V, Diode_SMD:D_MicroMELF_Handsoldering, F.Cu at (159.2, 55.1)
- added D5: 1N4007, Diode_SMD:D_SOD-123, F.Cu at (152.6, 55.6)
- added D6: B120-E3, Diode_SMD:D_SMA, F.Cu at (105.2, 107.7)
- added D7: 1N4007, Diode_SMD:D_SOD-123, F.Cu at (155.9, 55.6)
- added L1: 330uH, Inductor_SMD:L_Coilcraft_LPS3314, F.Cu at (136.8, 52.6)
- C8: footprint Capacitor_THT:C_Disc_D11.0mm_W5.0mm_P5.00mm -> Capacitor_SMD:C_0402_1005Metric
- U1: footprint Package_SO:SOIC-8_3.9x4.9mm_P1.27mm -> Package_SO:TSSOP-8_3x3mm_P0.65mm
- U3: value L7805 -> LM2596S-5; footprint Package_TO_SOT_THT:TO-220F-3_Vertical -> Package_TO_SOT_SMD:TO-263-5_TabPin3
- moved Iron_conect1 109.1 mm to (192.3, 55.0)
- moved C1 84.4 mm to (171.0, 110.6)
- moved J1 74.0 mm to (184.9, 55.6), turned to 180 degrees
- moved R14 62.1 mm to (155.6, 51.5), turned to 90 degrees
- moved R11 59.7 mm to (153.8, 51.5), turned to 90 degrees
- moved U2 57.8 mm to (161.1, 113.4)
- moved R7 57.3 mm to (152.1, 51.5), turned to 90 degrees
- moved R6 55.0 mm to (150.3, 51.5), turned to 90 degrees
- moved BZ1 54.6 mm to (80.6, 105.1)
- moved Q1 53.9 mm to (102.6, 102.8)
- moved R4 52.7 mm to (148.6, 51.5), turned to 90 degrees
- moved R3 50.3 mm to (146.8, 51.5), turned to 90 degrees
- moved R1 48.0 mm to (145.1, 51.5), turned to 90 degrees
- moved C8 46.6 mm to (171.0, 114.5)
- moved R5 41.2 mm to (117.6, 103.1)
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Connections:
- C8 pad 1: unconnected-(C8-Pad1) -> Net-(D2-A)
- C8 pad 2: unconnected-(C8-Pad2) -> GND
- J1 pad 2: 24V+ -> +24V
- R12 pad 1: 24V+ -> +24V
- U2 pad 2: 24V+ -> +24V
- U3 pad 1: 24V+ -> Net-(D5-K)
- U3 pad 2: GND -> Net-(D6-K)
- U3 pad 3: VCC -> GND
Routing:
- net GND: track 14.4 -> 296.2 mm
- net D9: track 0.00 -> 86.5 mm
- net D10: track 0.00 -> 48.6 mm
- net unconnected-(A1-SCK-Pad16): track 0.00 -> 41.2 mm
- net A0: track 0.00 -> 36.1 mm
- net Net-(D2-A): track 0.00 -> 35.5 mm
- net Net-(U1A--): track 0.00 -> 34.2 mm
- net D5: track 33.9 -> 0.00 mm
- net unconnected-(A1-~{RESET}-Pad28): track 0.00 -> 29.9 mm
- net unconnected-(A1-RX1-Pad2): track 0.00 -> 29.2 mm
- net Net-(U1B-+): track 0.00 -> 27.0 mm
- net B: track 0.00 -> 24.6 mm
- net A: track 0.00 -> 24.4 mm
- net Net-(D7-A): track 0.00 -> 13.4 mm
- net VCC: track 0.00 -> 11.1 mm
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- added copper zone on F.Cu, net GND
Other:
- board outline added: 147.2 x 69.3 mm

Commit message: update
Parts:
- removed Brd1: SSD1306, library:128x64OLED
- moved D6 62.9 mm to (162.1, 81.0)
- moved R8 61.8 mm to (172.9, 86.9)
- moved R9 61.8 mm to (172.9, 88.8)
- moved R5 58.2 mm to (172.9, 84.9)
- moved R12 57.8 mm to (134.5, 110.5), turned to 0 degrees
- moved D3 57.3 mm to (135.7, 107.4), turned to 0 degrees
- moved L1 56.3 mm to (129.7, 108.5), turned to 0 degrees
- moved C13 55.5 mm to (169.3, 106.5), turned to 0 degrees
- moved C7 52.0 mm to (169.3, 99.7), turned to 0 degrees
- moved R13 51.8 mm to (122.1, 111.8), turned to 0 degrees
- moved R14 46.1 mm to (170.2, 95.2), turned to 0 degrees
- moved R11 45.1 mm to (170.2, 93.5), turned to 0 degrees
- moved R7 44.2 mm to (170.2, 91.8), turned to 0 degrees
- moved R6 43.3 mm to (170.2, 90.0), turned to 0 degrees
- moved R4 42.7 mm to (170.2, 88.2), turned to 0 degrees
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Routing:
- net GND: track 296.2 -> 514.9 mm
- net VCC: track 11.1 -> 203.1 mm
- net unconnected-(A1-D3-Pad6): track 0.00 -> 73.9 mm
- net unconnected-(A1-D2-Pad5): track 0.00 -> 67.1 mm
- net Net-(D2-A): track 35.5 -> 101.9 mm
- net Net-(D6-K): track 0.00 -> 62.6 mm
- net Net-(D7-A): track 13.4 -> 75.8 mm
- net +24V: track 0.00 -> 62.1 mm
- net Net-(D5-K): track 0.00 -> 55.0 mm
- net D10: track 48.6 -> 0.00 mm
- net Net-(Q1-B): track 0.00 -> 46.3 mm
- net Net-(D1-K): track 0.00 -> 45.2 mm
- net unconnected-(A1-SCK-Pad16): track 41.2 -> 0.00 mm
- net A: track 24.4 -> 61.6 mm
- net A0: track 36.1 -> 0.00 mm
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- removed copper zone on F.Cu, net GND

Commit message: update
Parts:
- removed A1: Arduino_Nano_Every, Module:Arduino_Nano
- removed BZ1: Buzzer, Buzzer_Beeper:Buzzer_12x9.5RM7.6
- removed C1: 100nF, Capacitor_SMD:C_0402_1005Metric
- removed C13: 10µF, Capacitor_SMD:CP_Elec_5x4.4
- removed C3: 100nf, Capacitor_SMD:C_0402_1005Metric
- removed C4, C5: 220uf, Capacitor_SMD:CP_Elec_8x10
- removed C7: 10uf 35V, Capacitor_SMD:CP_Elec_5x4.4
- removed C8: 2nF, Capacitor_SMD:C_0402_1005Metric
- removed D1: 1N5819, Diode_SMD:D_SOD-123
- removed D2, D5, D7: 1N4007, Diode_SMD:D_SOD-123
- removed D3: 5V, Diode_SMD:D_MicroMELF_Handsoldering
- removed D4: 18v, Diode_SMD:D_MiniMELF_Handsoldering
- removed D6: B120-E3, Diode_SMD:D_SMA
- removed Iron_conect1: Conn_01x05_Pin, TerminalBlock_MetzConnect:TerminalBlock_MetzConnect_Type101_RT01605HBWC_1x05_P5.08mm_Horizontal
- removed J1: Conn_01x02_Pin, TerminalBlock_MetzConnect:TerminalBlock_MetzConnect_Type101_RT01602HBWC_1x02_P5.08mm_Horizontal
- removed L1: 330uH, Inductor_SMD:L_Coilcraft_LPS3314
- removed Q1: PN2222A, Package_TO_SOT_THT:TO-92_Wide
- removed R1, R11, R14, R3, R4, R6, R7: 10K, Resistor_SMD:R_0201_0603Metric
- removed R12: 47K, Resistor_SMD:R_0805_2012Metric
- removed R13: 10K, Resistor_SMD:R_0603_1608Metric
- removed R5: 4.7K, Resistor_SMD:R_0402_1005Metric
- removed R8: 200K, Resistor_SMD:R_0402_1005Metric
- removed R9: 1K, Resistor_SMD:R_0402_1005Metric
- removed SW1: RotaryEncoder_Switch_MP, Rotary_Encoder:RotaryEncoder_Alps_EC11E-Switch_Vertical_H20mm
- removed U1: LM358, Package_SO:TSSOP-8_3x3mm_P0.65mm
- removed U2: IRLIZ44N, Package_TO_SOT_THT:TO-220F-3_Vertical
- removed U3: LM2596S-5, Package_TO_SOT_SMD:TO-263-5_TabPin3
Routing:
- net GND: track 514.9 -> 0.00 mm
- net VCC: track 203.1 -> 0.00 mm
- net D9: track 104.0 -> 0.00 mm
- net Net-(D2-A): track 101.9 -> 0.00 mm
- net Net-(D7-A): track 75.8 -> 0.00 mm
- net unconnected-(A1-D3-Pad6): track 73.9 -> 0.00 mm
- net unconnected-(A1-D2-Pad5): track 67.1 -> 0.00 mm
- net Net-(D6-K): track 62.6 -> 0.00 mm
- net +24V: track 62.1 -> 0.00 mm
- net A: track 61.6 -> 0.00 mm
- net Net-(D5-K): track 55.0 -> 0.00 mm
- net Net-(Q1-B): track 46.3 -> 0.00 mm
- net Net-(D1-K): track 45.2 -> 0.00 mm
- net unconnected-(A1-MISO-Pad15): track 34.1 -> 0.00 mm
- net D5: track 29.6 -> 0.00 mm
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
Commit message: update
Parts:
- added A1: Arduino_Nano_Every, Module:Arduino_Nano, F.Cu at (128.9, 125.6)
- added BZ1: Buzzer, Buzzer_Beeper:Buzzer_12x9.5RM7.6, F.Cu at (90.5, 120.5)
- added Brd1: SSD1306, library:128x64OLED, B.Cu at (126.7, 102.0)
- added C1: 100nF, Capacitor_SMD:C_1206_3216Metric, F.Cu at (120.5, 120.5)
- added C13: 10uf 35V, Capacitor_SMD:CP_Elec_5x5.7, F.Cu at (138.6, 104.3)
- added C3: 100nf, Capacitor_SMD:C_1206_3216Metric, F.Cu at (129.4, 83.5)
- added C4: 220uf, Capacitor_SMD:CP_Elec_8x10, F.Cu at (145.8, 95.3)
- added C5: 220uf, Capacitor_SMD:CP_Elec_8x10, F.Cu at (129.8, 92.6)
- added C7: 10uf 35V, Capacitor_SMD:CP_Elec_5x5.7, F.Cu at (151.3, 104.5)
- added C8: 2nF, Capacitor_SMD:C_1206_3216Metric, F.Cu at (153.9, 129.9)
- added D1: 1N5819, Diode_SMD:D_SOD-123, F.Cu at (177.5, 123.5)
- added D2: 1N4007, Diode_SMD:D_SMA, F.Cu at (148.8, 128.4)
- added D3: 5V, Diode_SMD:D_MicroMELF_Handsoldering, F.Cu at (113.5, 96.3)
- added D4: 18v, Diode_SMD:D_MiniMELF_Handsoldering, F.Cu at (144.6, 113.1)
- added D5: 1N4007, Diode_SMD:D_SMA, F.Cu at (170.6, 122.3)
- added D6: SS34, Diode_SMD:D_SMA, F.Cu at (170.6, 126.9)
- added D7: 1N4007, Diode_SMD:D_SMA, F.Cu at (170.6, 131.4)
- added Iron_conect1: Conn_01x05_Pin, TerminalBlock_MetzConnect:TerminalBlock_MetzConnect_Type101_RT01605HBWC_1x05_P5.08mm_Horizontal, F.Cu at (89.4, 79.9)
- added J1: Conn_01x02_Pin, TerminalBlock_MetzConnect:TerminalBlock_MetzConnect_Type101_RT01602HBWC_1x02_P5.08mm_Horizontal, F.Cu at (116.4, 79.7)
- added Q1: 2N2222A, Package_TO_SOT_SMD:SOT-23_Handsoldering, F.Cu at (137.7, 140.2)
- added R1: 10K, Resistor_SMD:R_1206_3216Metric, F.Cu at (145.2, 121.3)
- added R11: 10K, Resistor_SMD:R_1206_3216Metric, F.Cu at (144.0, 133.7)
- added R12: 47K, Resistor_SMD:R_1206_3216Metric, F.Cu at (118.7, 92.4)
- added R13: 10K, Resistor_SMD:R_1206_3216Metric, F.Cu at (117.0, 96.3)
- added R14: 10K, Resistor_SMD:R_1206_3216Metric, F.Cu at (100.8, 87.0)
- added R3: 10K, Resistor_SMD:R_1206_3216Metric, F.Cu at (128.3, 117.0)
- added R4: 10K, Resistor_SMD:R_1206_3216Metric, F.Cu at (132.5, 117.0)
- added R5: 4.7K, Resistor_SMD:R_1206_3216Metric, F.Cu at (122.4, 108.9)
- added R6: 10K, Resistor_SMD:R_1206_3216Metric, F.Cu at (128.0, 99.0)
- added R7: 10K, Resistor_SMD:R_1206_3216Metric, F.Cu at (128.0, 102.3)
- added R8: 200K, Resistor_SMD:R_1206_3216Metric, F.Cu at (128.0, 105.6)
- added R9: 1K, Resistor_SMD:R_1206_3216Metric, F.Cu at (128.0, 108.9)
- added SW1: RotaryEncoder_Switch_MP, Rotary_Encoder:RotaryEncoder_Alps_EC11E-Switch_Vertical_H20mm, B.Cu at (107.2, 109.2)
- added U1: LM358, Package_SO:TSSOP-8_3x3mm_P0.65mm, F.Cu at (138.9, 119.3)
- added U2: IRLIZ44N, Package_TO_SOT_THT:TO-220F-3_Vertical, F.Cu at (152.0, 120.4)
- added U3: LM2596S-5, Package_TO_SOT_SMD:TO-263-5_TabPin3, F.Cu at (148.2, 81.7)
Other:
- board size 147.2 x 69.3 mm -> 70 x 70 mm
